File: hardware/main/pcie_analyzer/pcie_analyzer.kicad_pcb (KiCad board)
At the start: 2 copper layers, 61 x 77.1 mm, 50 parts, among them J1 HDR40, J2 HDR40, J3 Conn_Coaxial, J4 Conn_Coaxial, J5 Conn_Coaxial, J6 Conn_Coaxial, J7 Conn_Coaxial, J8 Conn_Coaxial

Commit message: placement components
Parts:
- moved C13 71.2 mm to (77.3, 34.5), turned to 270 degrees
- moved C1 69.0 mm to (83.6, 32.8), turned to 0 degrees
- moved C25 67.9 mm to (79.3, 31.2), turned to 270 degrees
- moved D3 66.4 mm to (95.2, 34.7), turned to 270 degrees
- moved C17 63.4 mm to (95.6, 30.6), turned to 180 degrees
- moved C21 63.0 mm to (92.2, 33.4), turned to 180 degrees
- moved C11 62.7 mm to (95.6, 31.8), turned to 180 degrees
- moved C12 62.4 mm to (92.2, 34.7), turned to 180 degrees
- moved C22 62.0 mm to (80.5, 31.2), turned to 270 degrees
- moved C27 59.2 mm to (98.3, 33.9), turned to 180 degrees
- moved FB1 56.1 mm to (74.9, 34.5), turned to 270 degrees
- moved C15 56.0 mm to (76.5, 49.8), turned to 270 degrees
- moved C18 54.5 mm to (92.2, 35.9), turned to 180 degrees
- moved D2 54.5 mm to (80.4, 49.9), turned to 0 degrees
- moved FB2 53.6 mm to (75.3, 49.8), turned to 270 degrees
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Connections:
- net Net-(D2-Pad10) renamed LOS2
- net Net-(D3-Pad10) renamed LOS3
- D1 pad 1: LOS1 -> Net-(C13-Pad1)
- D1 pad 10: Net-(D1-Pad10) -> LOS1
- D1 pad 2: LOS1 -> Net-(C13-Pad1)
- D2 pad 1: LOS1 -> Net-(C15-Pad1)
- D2 pad 2: LOS1 -> Net-(C15-Pad1)
- D3 pad 1: LOS1 -> Net-(C11-Pad1)
- D3 pad 2: LOS1 -> Net-(C11-Pad1)
- FB1 pad 2: LOS1 -> +3.3VCC
- FB2 pad 2: LOS1 -> +3.3VCC
- FB3 pad 2: LOS1 -> +3.3VCC
- J1 pad 25: LOS1 -> +3.3VCC
- J1 pad 27: LOS1 -> +3.3VCC
- J1 pad 35: LOS1 -> +3.3VCC
- J1 pad 37: LOS1 -> +3.3VCC
- J1 pad 39: LOS1 -> +3.3VCC
- J2 pad 20: LOS1 -> +3.3VCC
- R7 pad 1: Net-(D1-Pad10) -> LOS1
- R7 pad 2: LOS1 -> +3.3VCC
- R8 pad 2: LOS1 -> +3.3VCC
- R9 pad 2: LOS1 -> +3.3VCC
Other:
- board size 61 x 77.1 mm -> 48 x 85 mm

Commit message: pcb work
Parts:
- added ST1: AXIAL_CABLE_SL8800_08, ecp5_pcie_analyzer:AXIAL_CABLE_SL8800_08, F.Cu at (93.2, 71.3)
- moved J5 33.6 mm to (102.9, 27.7)
- moved J8 30.0 mm to (73.0, 43.3)
- moved J7 29.9 mm to (73.1, 28.1)
- moved C27 22.2 mm to (76.3, 36.2), turned to 0 degrees
- moved R6 22.2 mm to (76.3, 33.8), turned to 0 degrees
- moved C24 22.1 mm to (76.3, 35.0), turned to 0 degrees
- moved C13 21.5 mm to (93.0, 49.3)
- moved C7 21.5 mm to (91.8, 49.3)
- moved C8 21.5 mm to (95.8, 52.8)
- moved FB1 21.5 mm to (90.6, 49.3)
- moved R1 21.5 mm to (99.3, 51.1)
- moved R7 21.5 mm to (99.3, 49.9)
- moved C14 21.5 mm to (97.0, 52.8)
- moved C19 21.5 mm to (94.4, 52.8)
- moved C4 21.5 mm to (99.2, 48.7)
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Routing:
- net PCIE_UP_P: track 0.00 -> 3.44 mm
- net PCIE_UP_N: track 0.00 -> 3.44 mm
Other:
- board size 48 x 85 mm -> 50 x 85 mm
- copper layers 2 -> 4
- net class Default: clearance 0.2 -> 0.2032; trace_width 0.25 -> 0.205232; via_dia 0.8 -> 0.6; via_drill 0.4 -> 0.2
- net class Diff added: clearance 0.2032, trace_width 0.205232, via_dia 0.6, via_drill 0.2
- rule trace_clearance: 0.2 -> 0.2032
- rule trace_min: 0.2 -> 0.1
- rule via_min_drill: 0.3 -> 0.2
- board text added: "103"
- board text added: "28"
- board text added: "43"
- board text added: "73"
- board text added: "88"

Commit message: daily work
Parts:
- moved ST1 4.60 mm to (93.8, 66.8)
- moved C10 1.73 mm to (95.7, 39.0)
- moved C20 1.72 mm to (94.5, 39.0)
- moved C16 1.71 mm to (96.8, 39.0)
- moved C18 1.59 mm to (84.0, 34.5)
- moved C12 1.57 mm to (84.0, 35.6)
- moved C21 1.57 mm to (84.0, 36.8)
- moved C11 1.31 mm to (80.3, 38.5)
- moved FB3 1.30 mm to (80.3, 40.6)
- moved C17 1.29 mm to (80.3, 39.5)
- moved C14 1.27 mm to (96.5, 54.0)
- moved D2 1.24 mm to (95.5, 35.5)
- moved C8 1.23 mm to (95.5, 54.0)
- moved C13 1.21 mm to (92.5, 50.4)
- moved C19 1.20 mm to (94.2, 54.0)
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Connections:
- J1 pad 11: Net-(J1-Pad11) -> DISABLE1
- J1 pad 13: Net-(J1-Pad13) -> DISABLE2
- J1 pad 15: Net-(J1-Pad15) -> DISABLE_CLK
- ST1 pad 1: PCIE_UP_P -> PCIE_DOWN_P
- ST1 pad 2: PCIE_UP_N -> PCIE_DOWN_N
- ST1 pad 3: PCIE_DOWN_P -> PCIE_UP_P
- ST1 pad 4: PCIE_DOWN_N -> PCIE_UP_N
Routing:
- net DISABLE2: track 0.00 -> 64.3 mm, vias 0 -> 1
- net CLK_P: track 0.00 -> 57.3 mm
- net CLK_N: track 0.00 -> 56.6 mm
- net LOS2: track 0.00 -> 52.9 mm, vias 0 -> 1
- net LOS1: track 0.00 -> 51.6 mm, vias 0 -> 1
- net DISABLE_CLK: track 0.00 -> 48.9 mm, vias 0 -> 1
- net DISABLE1: track 0.00 -> 47.6 mm, vias 0 -> 1
- net PCIE_DOWN_N: track 0.00 -> 44.5 mm, vias 0 -> 2
- net PCIE_DOWN_P: track 0.00 -> 43.0 mm, vias 0 -> 2
- net LOS3: track 0.00 -> 39.6 mm, vias 0 -> 1
- net PCIE_UP_N: track 3.44 -> 33.4 mm
- net PCIE_UP_P: track 3.44 -> 31.9 mm
- net PCIE_1_N: track 0.00 -> 9.22 mm
- net PCIE_2_N: track 0.00 -> 9.20 mm
- net PCIE_CLK_N: track 0.00 -> 9.20 mm
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- added copper zone on In2.Cu, net +3.3VCC
- added copper zone on F.Cu, net GND
- added copper zone on In1.Cu, net GND
Other:
- net class Single endet 50 added: clearance 0.3, trace_width 0.29337, via_dia 0.6, via_drill 0.2

Commit message: pcb work
Parts:
- moved C10 1.67 mm to (97.3, 39.2), turned to 0 degrees
- moved C16 1.11 mm to (97.4, 38.1), turned to 0 degrees
- moved C20 0.23 mm to (94.2, 39.0)
Connections:
- J1 pad 11: DISABLE1 -> LOS2
- J1 pad 13: DISABLE2 -> DISABLE1
- J1 pad 15: DISABLE_CLK -> LOS1
- J1 pad 5: LOS1 -> DISABLE_CLK
- J1 pad 7: LOS2 -> LOS3
- J1 pad 9: LOS3 -> DISABLE2
Routing:
- net GND: track 5.90 -> 23.4 mm, vias 7 -> 26
- net DISABLE_CLK: track 48.9 -> 31.6 mm
- net LOS1: track 51.6 -> 36.3 mm
- net PCIE_DOWN_N: track 44.5 -> 59.1 mm, vias 2 -> 0
- net PCIE_DOWN_P: track 43.0 -> 57.1 mm, vias 2 -> 0
- net DISABLE2: track 64.3 -> 52.1 mm
- net DISABLE1: track 47.6 -> 39.4 mm
- net LOS3: track 39.6 -> 31.6 mm
- net PCIE_UP_N: track 33.4 -> 27.3 mm
- net PCIE_UP_P: track 31.9 -> 26.0 mm
- net LOS2: track 52.9 -> 49.0 mm
- net CLK_P: track 57.3 -> 54.8 mm
- net CLK_N: track 56.6 -> 54.1 mm
- net Net-(C10-Pad1): track 1.62 -> 2.93 mm
- net +3.3VCC: track 4.46 -> 4.12 mm, vias 5 -> 6
- added copper zone on B.Cu, net GND
Other:
- net class Default: trace_width 0.205232 -> 0.2; via_dia 0.6 -> 0.4

Commit message: first release sch/pcb
Parts:
- added R10: 0, ecp5_pcie_analyzer:R_0402, F.Cu at (81.2, 63.0)
- added R11: 0, ecp5_pcie_analyzer:R_0402, F.Cu at (95.7, 62.8)
- moved C11 0.17 mm to (80.3, 38.3)
- moved C3 0.15 mm to (78.3, 32.0)
- moved C14 0.13 mm to (96.6, 54.0)
- moved R5 0.13 mm to (97.2, 32.0)
- moved C27 0.12 mm to (77.0, 36.2)
- moved FB2 0.12 mm to (90.2, 35.3)
- moved FB1 0.12 mm to (90.3, 50.4)
- moved C13 0.12 mm to (92.6, 50.4)
- moved C26 0.12 mm to (94.9, 32.0)
- moved R6 0.11 mm to (77.0, 33.9)
- moved C6 0.08 mm to (79.5, 32.0)
- moved R8 0.07 mm to (99.0, 35.7)
- moved C9 0.07 mm to (92.6, 35.3)
- moved C25 0.07 mm to (94.8, 47.0)
- moved R4 0.07 mm to (97.2, 47.0)
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Routing:
- net GND: track 23.4 -> 253.7 mm, vias 26 -> 110
- net Net-(R11-Pad1): track 0.00 -> 3.90 mm
- net Net-(R10-Pad1): track 0.00 -> 3.32 mm
Other:
- outline, holes or cut-outs redrawn
- board text added: "1"
- board text added: "2"
- board text added: "3"
- board text added: "4"
- board text added: "CLK_N"
- board text added: "CLK_P"
- board text added: "RX1_N"
- board text added: "RX1_P"
- board text added: "RX2_N"
- board text added: "RX2_P"
- board text added: "V1"
